File: hardware/node/node.kicad_pcb (KiCad board)
At the start: 2 copper layers, 27.1 x 45 mm, 47 parts, among them J1 USB_C_Receptacle_USB2.0_14P, J2 SWD, J3 Batt, J4 Solar, Q1 8205A_C2762931, U1 VGDD79S868N0S1, U2 MS88SF3-NRF52840, U3 SRV05-4, U4 TP4056-42-ESOP8, U5 DW01A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

Commit message: routing
Parts:
- added F2: Polyfuse, Fuse:Fuse_0603_1608Metric, F.Cu at (134.9, 110.1)
- added R12: 0r, Resistor_SMD:R_0603_1608Metric, F.Cu at (136.8, 107.9)
- added TP2: TestPoint, TestPoint:TestPoint_Pad_1.5x1.5mm, F.Cu at (135.1, 112.2)
- added TP3: TestPoint, TestPoint:TestPoint_Pad_1.5x1.5mm, F.Cu at (129.4, 118.7)
- added TP4: TestPoint, TestPoint:TestPoint_Pad_1.5x1.5mm, F.Cu at (131.9, 118.7)
- added TP5: TestPoint, TestPoint:TestPoint_Pad_1.5x1.5mm, F.Cu at (142.1, 103.5)
- F1: footprint Capacitor_SMD:C_0603_1608Metric_Pad1.08x0.95mm_HandSolder -> Fuse:Fuse_0603_1608Metric
- moved R3 6.28 mm to (140.5, 114.8)
- moved R1 2.41 mm to (138.1, 114.9)
- moved C8 1.46 mm to (140.5, 107.1)
- moved R2 1.46 mm to (139.0, 107.1)
- moved C18 1.46 mm to (147.5, 119.4)
- moved R11 1.46 mm to (146.0, 119.4)
- moved Q1 1.32 mm to (128.6, 101.8)
- moved U3 1.04 mm to (138.2, 110.7)
- moved D3 0.63 mm to (146.2, 104.4)
Connections:
- U2 pad 29: unconnected-(U2-P0.16-Pad29) -> /scl
- U2 pad 30: unconnected-(U2-P0.14-Pad30) -> /sdl
Routing:
- net VBUS: track 0.00 -> 58.1 mm, vias 0 -> 3
- net +BATT: track 0.00 -> 55.0 mm
- net /d-: track 0.00 -> 27.9 mm, vias 0 -> 2
- net Net-(J2-Pin_2): track 0.00 -> 22.0 mm, vias 0 -> 1
- net /d+: track 0.00 -> 21.6 mm
- net Net-(J2-Pin_3): track 0.00 -> 20.1 mm, vias 0 -> 1
- net +3V3: track 0.00 -> 19.7 mm
- net -BATT: track 0.00 -> 16.2 mm
- net /dio3: track 0.00 -> 14.4 mm
- net +6V: track 0.00 -> 13.5 mm
- net /sdl: track 0.00 -> 13.0 mm, vias 0 -> 2
- net /cs: track 0.00 -> 12.3 mm
- net Net-(U2-VBUS): track 0.00 -> 11.9 mm
- net /scl: track 0.00 -> 11.6 mm, vias 0 -> 2
- net /dio1: track 0.00 -> 11.5 mm
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- added copper zone on B.Cu, net GND
- added copper zone on F.Cu, net GND

Commit message: ufl  antenna
Parts:
- added AE1: U.FL, Connector_Coaxial:U.FL_Hirose_U.FL-R-SMT-1_Vertical, F.Cu at (130.4, 137.2)
- added C20: c, Capacitor_SMD:C_0402_1005Metric, F.Cu at (133.2, 136.7)
- added L2: L, Inductor_SMD:L_0402_1005Metric, F.Cu at (134.4, 135.2)
Routing:
- net +BATT: track 55.0 -> 68.0 mm, vias 0 -> 2
- net Net-(AE1-A): track 0.00 -> 4.15 mm
- net /antenna: track 0.00 -> 1.35 mm

Commit message: uuuu
Parts:
- D2: value (insert 5v clamp voltage) -> TPGC03C-A; footprint Diode_THT:D_DO-201AE_P15.24mm_Horizontal -> Diode_SMD:D_SOD-323
- R10, R11: value 1m -> 1M
- moved D2 98.5 mm to (136.9, 117.8), turned to -90 degrees
- moved C15 0.86 mm to (143.7, 118.7)
- moved C3 0.86 mm to (138.6, 117.9)
- moved C4 0.86 mm to (140.1, 117.9)
- moved C5 0.86 mm to (141.5, 117.9)
- moved R1 0.54 mm to (138.6, 114.9)
Routing:
- net +BATT: track 68.0 -> 69.8 mm
- net /batt_sens: track 9.24 -> 7.86 mm
- net GND: vias 77 -> 98
Other:
- outline, holes or cut-outs redrawn

Commit message: push before fork
Parts:
- moved D1 0.35 mm to (134.3, 101.9)
- moved R6 0.33 mm to (137.5, 101.9)
- moved U4 0.23 mm to (140.2, 98.4)
- moved U7 0.23 mm to (140.2, 98.4)
- moved R2 0.08 mm to (139.0, 107.2)
- moved U3 0.08 mm to (138.2, 110.7)
Other:
- board text added: "swclk"
- board text added: "swdio"

Commit message: a
Parts:
- removed C10, C11, C12, C13, C15, C4, C5: 10u, Capacitor_SMD:C_0603_1608Metric
- removed C14, C18, C3, C8: 100n, Capacitor_SMD:C_0603_1608Metric
- removed D2: TPGC03C-A, Diode_SMD:D_SOD-323
- removed D3: 1N4148W, Diode_SMD:D_SOD-123
- removed F2: Polyfuse, Fuse:Fuse_0603_1608Metric
- removed J2: SWD, Connector_PinHeader_2.54mm:PinHeader_1x04_P2.54mm_Vertical
- removed L1: 10u 80ma+, Inductor_SMD:L_0603_1608Metric
- removed R1, R2: 5.1k, Resistor_SMD:R_0603_1608Metric
- removed R10, R11, R9: 1M, Resistor_SMD:R_0603_1608Metric
- removed R12, R3: 0r, Resistor_SMD:R_0603_1608Metric
- removed TP2, TP3, TP4, TP5: TestPoint, TestPoint:TestPoint_Pad_1.5x1.5mm
- removed U3: SRV05-4, Package_TO_SOT_SMD:SOT-23-6
- removed U6: ME6217C33M5G, Package_TO_SOT_SMD:SOT-23-5
- J1: value USB_C_Receptacle_USB2.0_14P -> Conn_01x04; footprint Connector_USB:USB_C_Receptacle_G-Switch_GT-USB-7010ASV -> Connector_PinHeader_2.54mm:PinHeader_1x04_P2.54mm_Vertical
- U2: value MS88SF3-NRF52840 -> nice_nano; footprint easyeda2kicad:BULETM-SMD_MS88SF3_V1.0 -> library:SuperMini NRF52840
- moved U2 71.2 mm to (213.6, 138.3)
- moved C16 65.4 mm to (210.3, 97.8)
- moved R5 65.4 mm to (210.3, 97.8)
- moved R7 65.4 mm to (210.3, 100.8)
- moved C17 65.4 mm to (201.0, 96.8)
- moved C9 65.4 mm to (199.5, 96.8)
- moved D1 65.4 mm to (199.8, 102.0)
- moved J4 65.4 mm to (213.2, 97.3)
- moved R6 65.4 mm to (202.9, 102.1)
- moved R8 65.4 mm to (201.0, 99.8)
- moved U4 65.4 mm to (205.7, 98.6)
- moved U7 65.4 mm to (205.7, 98.6)
- moved C6 60.9 mm to (194.5, 106.1)
- moved F1 60.9 mm to (189.5, 97.2)
- moved Q1 60.9 mm to (189.4, 101.8)
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Connections:
- U2 pad 1: GND -> /sdl
- U2 pad 10: unconnected-(U2-P0.29-Pad10) -> /dio3
- U2 pad 13: unconnected-(U2-P0.31-Pad13) -> +BATT
- U2 pad 14: unconnected-(U2-P0.27-Pad14) -> GND
- U2 pad 15: /batt_sens -> unconnected-(U2-RST-Pad15)
- U2 pad 16: unconnected-(U2-P0.04-Pad16) -> +3V3
- U2 pad 17: unconnected-(U2-P0.26-Pad17) -> /busy
- U2 pad 18: GND -> unconnected-(U2-P0.29-Pad18)
- U2 pad 19: unconnected-(U2-P0.07-Pad19) -> /rst
- U2 pad 2: unconnected-(U2-P1.11-Pad2) -> /scl
- U2 pad 28: unconnected-(U2-P0.18-Pad28) -> GND
- U2 pad 29: /scl -> +BATT
- U2 pad 3: unconnected-(U2-P1.12-Pad3) -> GND
- U2 pad 4: unconnected-(U2-P1.10-Pad4) -> GND
- U2 pad 5: unconnected-(U2-P1.14-Pad5) -> /cs
- U2 pad 6: unconnected-(U2-P0.03-Pad6) -> /clk
- U2 pad 7: unconnected-(U2-P1.13-Pad7) -> /mosi
- U2 pad 8: unconnected-(U2-P1.15-Pad8) -> /miso
- U2 pad 9: unconnected-(U2-P0.02-Pad9) -> /dio1
Routing:
- net VBUS: track 58.5 -> 0.00 mm, vias 3 -> 0
- net /d-: track 28.3 -> 0.00 mm, vias 2 -> 0
- net /dio3: track 14.4 -> 36.6 mm, vias 0 -> 1
- net /d+: track 22.0 -> 0.00 mm
- net Net-(J2-Pin_2): track 22.0 -> 0.00 mm, vias 1 -> 0
- net /scl: track 11.6 -> 33.6 mm, vias 2 -> 1
- net /dio1: track 11.5 -> 32.3 mm, vias 0 -> 1
- net Net-(J2-Pin_3): track 20.1 -> 0.00 mm, vias 1 -> 0
- net /sdl: track 13.0 -> 32.9 mm, vias 2 -> 1
- net /miso: track 6.63 -> 21.9 mm
- net /mosi: track 8.43 -> 23.3 mm
- net /clk: track 10.4 -> 25.0 mm
- net /cs: track 12.3 -> 26.7 mm
- net Net-(U2-VBUS): track 12.4 -> 0.00 mm
- net -BATT: track 16.2 -> 24.9 mm, vias 0 -> 1
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Other:
- board size 27.1 x 45 mm -> 31.7 x 45 mm
- board text removed: "swclk"
- board text removed: "swdio"

Commit message: a
Parts:
- removed C9: 10u, Capacitor_SMD:C_0603_1608Metric
- removed D1: LED, Capacitor_SMD:C_0603_1608Metric_Pad1.08x0.95mm_HandSolder
- removed R5: 10r, Resistor_SMD:R_0603_1608Metric
- removed R6: 1k, Resistor_SMD:R_0603_1608Metric
- removed U4: TP4056-42-ESOP8, Package_SO:SOIC-8-1EP_3.9x4.9mm_P1.27mm_EP2.41x3.3mm_ThermalVias
Routing:
- net /chrg: track 7.55 -> 0.00 mm, vias 1 -> 0
- net +BATT: track 77.8 -> 74.7 mm, vias 2 -> 1
- net Net-(U7-FB): track 0.00 -> 2.25 mm
- net Net-(D1-K): track 1.45 -> 0.00 mm
Other:
- outline, holes or cut-outs redrawn
