File: hardware/node/node.kicad_sch (KiCad schematic)
At the start: 35 parts, among them J1 USB_C_Receptacle_USB2.0_14P, J2 SWD, J3 Batt, Q1 8205A_C2762931, U1 VGDD79S868N0S1, U2 MS88SF3-NRF52840, U3 SRV05-4, U4 TP4056-42-ESOP8, U5 DW01A, U6 AMS1117-3.3

Commit message: pcbbbb placement of parts etc
Parts:
- removed U6: AMS1117-3.3, Package_TO_SOT_SMD:SOT-223-3_TabPin2, symbol Regulator_Linear:AMS1117-3.3
- added C16, C17: 10u, Capacitor_SMD:C_0603_1608Metric, symbol Device:C
- added C18: 100n, Capacitor_SMD:C_0603_1608Metric, symbol Device:C
- added D3: 1N4148W, Diode_SMD:D_SOD-123, symbol Diode:1N4148W
- added J4: Solar, Connector_PinHeader_2.54mm:PinHeader_1x02_P2.54mm_Vertical, symbol Connector_Generic:Conn_01x02
- added L1: 10u 80ma+, Inductor_SMD:L_0603_1608Metric, symbol Device:L
- added R10, R11: 1m, Resistor_SMD:R_0603_1608Metric, symbol Device:R
- added R7: 1k, Resistor_SMD:R_0603_1608Metric, symbol Device:R
- added R8: 0r, Resistor_SMD:R_0603_1608Metric, symbol Device:R
- added R9: 1M, Resistor_SMD:R_0603_1608Metric, symbol Device:R
- added U6: ME6217C33M5G, Package_TO_SOT_SMD:SOT-23-5, symbol Regulator_Linear:ME6211C33M5
- added U7: CN3163, Package_SO:SOIC-8-1EP_3.9x4.9mm_P1.27mm_EP2.41x3.3mm_ThermalVias, symbol Battery_Management:CN3163
- C1, C10, C11, C12, C13, C14, C15, C2, C3, C4, C5, C6, C7, C8: footprint (none) -> Capacitor_SMD:C_0603_1608Metric
- C9: footprint (none) -> Capacitor_SMD:C_0603_1608Metric; now not fitted; now left out of the parts list
- D1, F1: footprint (none) -> Capacitor_SMD:C_0603_1608Metric_Pad1.08x0.95mm_HandSolder
- J1: footprint (none) -> Connector_USB:USB_C_Receptacle_G-Switch_GT-USB-7010ASV
- J2: footprint (none) -> Connector_PinHeader_2.54mm:PinHeader_1x04_P2.54mm_Vertical
- J3: footprint (none) -> Connector_PinHeader_2.54mm:PinHeader_1x03_P2.54mm_Vertical
- R1, R2, R3, R4, R6: footprint (none) -> Resistor_SMD:R_0603_1608Metric
- R5: footprint (none) -> Resistor_SMD:R_0603_1608Metric; now not fitted; now left out of the parts list
- TP1: footprint (none) -> TestPoint:TestPoint_Pad_1.5x1.5mm
- U4: now not fitted; now left out of the parts list
Connections:
- net +3V3: now also U6.5 (V_{OUT})
- net +BATT: now also C6.1, R4.1, C17.1, R10.1, R8.1, R9.2, U6.1 (V_{IN}), U7.5 (BAT)
- net GND: now also C16.2, C17.2, C18.2, J4.2 (Pin_2), R11.2, R7.2, U6.2 (V_{SS}), U7.1 (TEMP), U7.3 (GND), U7.9 (GND)
- net VBUS: now also D3.2 (A)
- net busy: now also U2.45 (P0.22)
- net clk: now also U2.41 (P0.17)
- net cs: now also U2.42 (P0.21)
- net d+: now also U3.6 (IO4); no longer U3.4 (IO3)
- net dio1: now also U2.44 (P0.20)
- net dio3: now also U2.43 (P0.23)
- net miso: now also U2.39 (P0.13)
- net mosi: now also U2.40 (P0.15)
- net rst: now also U2.38 (P0.19)
- net VCC: now reaches C14.1, C15.1, U2.31 (VDD)
- net VCC: now also L1.1
- net batt_sens: now reaches U2.15 (P0.05)
- net batt_sens: now also C18.1, R10.2, R11.1
- net at U2.33 (DCCH): now also L1.2
- net chrg: now reaches R6.2, U4.7 (~{CHRG})
- net chrg: now also U7.7 (~{CHRG})
- new net: R9.1, U6.3 (CE)
- new net: R8.2, U7.8 (FB)
- new net: R7.1, U7.2 (ISET)
- new net +6V: C16.1, D3.1 (K), J4.1 (Pin_1), U7.4 (VIN)
- no-connect marks 5 -> 6
Other:
- note added: "5Vin"
- note added: "VREG ＝ 4.2＋3.707×10-6×Rx if vreg = 4.2 then rx = 0 adjust for higher voltage batt"
- note added: "datasheet Riset = 1.18k for 1a @ 3.6v so 1k should be enough to make use of max charging power"
- moved on the sheet: C10, C11, C12, C13, C3, C4, C5, C8, D2, F1, J3

Commit message: routing
Parts:
- added C19: 10u, Capacitor_SMD:C_0603_1608Metric, symbol Device:C
- added F2: Polyfuse, Fuse:Fuse_0603_1608Metric, symbol Device:Polyfuse
- added R12: 0r, Resistor_SMD:R_0603_1608Metric, symbol Device:R
- added TP2, TP3, TP4, TP5: TestPoint, TestPoint:TestPoint_Pad_1.5x1.5mm, symbol Connector:TestPoint
- F1: footprint Capacitor_SMD:C_0603_1608Metric_Pad1.08x0.95mm_HandSolder -> Fuse:Fuse_0603_1608Metric
Connections:
- net +3V3: now also C19.1, F2.1
- net +BATT: now also R12.1
- net GND: now also C19.2, TP5.1
- net VBUS: now also R12.2
- net scl: now reaches U2.29 (P0.16)
- net scl: now also TP4.1
- net sdl: now reaches U2.30 (P0.14)
- net sdl: now also TP3.1
- new net: F2.2, TP2.1
- no-connect marks 6 -> 47
Other:
- moved on the sheet: C1, C2, U1

Commit message: ufl  antenna
Parts:
- added AE1: U.FL, Connector_Coaxial:U.FL_Hirose_U.FL-R-SMT-1_Vertical, symbol Device:Antenna_Shield
- added C20: c, Capacitor_SMD:C_0402_1005Metric, symbol Device:C
- added L2: L, Inductor_SMD:L_0402_1005Metric, symbol Device:L
Connections:
- net GND: now also AE1.2 (Shield), C20.2
- net antenna: now also L2.1
- new net: AE1.1 (A), C20.1, L2.2
Other:
- note added: "antenna L/C network"

Commit message: uuuu
Parts:
- AE1: LCSC Part (none) -> C88374
- C1, C14, C18, C3, C6, C7, C8: LCSC Part (none) -> C24497
- C10, C11, C12, C13, C15, C16, C17, C19, C2, C4, C5, C9: LCSC Part (none) -> C962136
- C20, J2, J3, J4, R5, TP1, TP2, TP3, TP4, TP5, U4: LCSC Part (none) -> x
- D1: LCSC Part (none) -> C965799
- D2: value (insert 5v clamp voltage) -> TPGC03C-A; footprint Diode_THT:D_DO-201AE_P15.24mm_Horizontal -> Diode_SMD:D_SOD-323; LCSC Part (none) -> C2827620
- D3: LCSC Part (none) -> C2099
- F1, F2: LCSC Part (none) -> C49318281
- J1: LCSC Part (none) -> C963411
- L2: LCSC Part (none) -> C242160
- R1, R2: LCSC Part (none) -> C123727
- R10, R11: value 1m -> 1M; LCSC Part (none) -> C407640
- R4: LCSC Part (none) -> C105588
- R6, R7: LCSC Part (none) -> C7422246
- R9: LCSC Part (none) -> C407640
- U3: LCSC Part (none) -> C151305
- U6: LCSC Part (none) -> C427602
- U7: LCSC Part (none) -> C559031

Commit message: push before fork
Other:
- note added: "USB"
- note added: "volatege divider"
- moved on the sheet: C18, C9, D1, L1, R10, R11, R3, R5, R6, U3, U4

Commit message: a
Parts:
- removed C10, C11, C12, C13, C15, C4, C5: 10u, Capacitor_SMD:C_0603_1608Metric, symbol Device:C
- removed C14, C18, C3, C8: 100n, Capacitor_SMD:C_0603_1608Metric, symbol Device:C
- removed D2: TPGC03C-A, Diode_SMD:D_SOD-323, symbol Diode:1.5KExxA
- removed D3: 1N4148W, Diode_SMD:D_SOD-123, symbol Diode:1N4148W
- removed J1: USB_C_Receptacle_USB2.0_14P, Connector_USB:USB_C_Receptacle_G-Switch_GT-USB-7010ASV, symbol Connector:USB_C_Receptacle_USB2.0_14P
- removed J2: SWD, Connector_PinHeader_2.54mm:PinHeader_1x04_P2.54mm_Vertical, symbol Connector_Generic:Conn_01x04
- removed L1: 10u 80ma+, Inductor_SMD:L_0603_1608Metric, symbol Device:L
- removed R1, R2: 5.1k, Resistor_SMD:R_0603_1608Metric, symbol Device:R
- removed R10, R11, R9: 1M, Resistor_SMD:R_0603_1608Metric, symbol Device:R
- removed R12, R3: 0r, Resistor_SMD:R_0603_1608Metric, symbol Device:R
- removed TP2, TP3, TP4, TP5: TestPoint, TestPoint:TestPoint_Pad_1.5x1.5mm, symbol Connector:TestPoint
- removed U2: MS88SF3-NRF52840, easyeda2kicad:BULETM-SMD_MS88SF3_V1.0, symbol easyeda2kicad:MS88SF3-NRF52840
- removed U3: SRV05-4, Package_TO_SOT_SMD:SOT-23-6, symbol Power_Protection:SRV05-4
- removed U6: ME6217C33M5G, Package_TO_SOT_SMD:SOT-23-5, symbol Regulator_Linear:ME6211C33M5
- added J1: Conn_01x04, Connector_PinHeader_2.54mm:PinHeader_1x04_P2.54mm_Vertical, symbol Connector_Generic:Conn_01x04
- added U2: nice_nano, library:SuperMini NRF52840, symbol nice_nano:nice_nano
- C19: now in the parts list
- R8: LCSC Part (none) -> x
Connections:
- net +3V3: now also U2.16 (3V3)
- net +BATT: now also U2.13 (batt+), U2.29 (batt+)
- net GND: now also J1.4 (Pin_4), U2.14 (GND), U2.28 (GND), U2.3 (GND), U2.4 (GND)
- net busy: now also U2.17 (P0.31)
- net clk: now also U2.6 (P0.20)
- net cs: now also U2.5 (P0.17)
- net dio1: now also U2.9 (P1.00)
- net dio3: now also U2.10 (P0.11)
- net miso: now also U2.8 (P0.24)
- net mosi: now also U2.7 (P0.22)
- net rst: now also U2.19 (P0.02)
- net scl: now also J1.3 (Pin_3), U2.2 (RX1/P0.08)
- net sdl: now also J1.2 (Pin_2), U2.1 (TX0/P0.06)
- net at F2.2: now also J1.1 (Pin_1)
- no-connect marks 47 -> 15
Other:
- note removed: "Decoupling and protection"
- note removed: "ESD"
- note removed: "USB"
- note removed: "debug"
- note removed: "power converter"
- note removed: "vddh abs rating 5.8v"
- note removed: "volatege divider"

Commit message: a
Parts:
- removed C9: 10u, Capacitor_SMD:C_0603_1608Metric, symbol Device:C
- removed D1: LED, Capacitor_SMD:C_0603_1608Metric_Pad1.08x0.95mm_HandSolder, symbol Device:LED
- removed R5: 10r, Resistor_SMD:R_0603_1608Metric, symbol Device:R
- removed R6: 1k, Resistor_SMD:R_0603_1608Metric, symbol Device:R
- removed U4: TP4056-42-ESOP8, Package_SO:SOIC-8-1EP_3.9x4.9mm_P1.27mm_EP2.41x3.3mm_ThermalVias, symbol Battery_Management:TP4056-42-ESOP8
Connections:
- net chrg: no longer names the net of U7.7 (~{CHRG})
- no-connect marks 15 -> 16
Other:
- note added: "display conn"
- note added: "mcu"
- note removed: "Charging circuit (~500ma)"
- note removed: "Ibat = (Vprog / Rprog) * 1100 Ibat = 500 Vprog = 5v (vcc limit of 3uA) 500 = 5500/Rprog Rprog * 500 = 5500 Rprog = 5500/500 Rprog = 11r"
- note removed: "datasheet Riset = 1.18k for 1a @ 3.6v so 1k should be enough to make use of max charging power"
- moved on the sheet: AE1, C1, C16, C17, C19, C2, C20, C6, C7, F1, F2, J1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
